File: example/nucleo-f767zi_solax-pylontech/pcb/Solax_Pylontech.kicad_sch (KiCad schematic)
At the start: 37 parts, among them J1 Conn_02x10_Odd_Even, J2 Conn_02x07_Odd_Even, U1 LT1107CS, U2 MCP2551-I-SN, U3 MCP2551-I-SN

Commit message: - implement battery balancing using external charger in front of each pack (HDR-15-48), each one driven by a triac module (MRA-23D2) - add home assistant shenanigans to drive the battery balancing (manual or automatic)
Parts:
- removed JI2CMON1, JUARTINV1: RJ45, Connector_RJ:RJ45_Amphenol_54602-x08_Horizontal, symbol Connector:RJ45
- added D6, D7: D_TVS, Diode_SMD:D_0603_1608Metric, symbol Device:D_TVS
- added H1, H2, H3: MountingHole, MountingHole:MountingHole_3mm, symbol Mechanical:MountingHole
- added J3: Conn_01x03_Socket, Connector_JST:JST_XH_B3B-XH-A_1x03_P2.50mm_Vertical, symbol Connector:Conn_01x03_Socket
- added J4: Conn_01x02_Socket, Connector_JST:JST_XH_B2B-XH-A_1x02_P2.50mm_Vertical, symbol Connector:Conn_01x02_Socket
- added J5, J6, J7, J8: Conn_01x05_Socket, Connector_JST:JST_XH_B5B-XH-A_1x05_P2.50mm_Vertical, symbol Connector:Conn_01x05_Socket
- added JUARTINV1: USB_C_Receptacle_USB2.0_16P, Connector_USB:USB_C_Receptacle_GCT_USB4105-xx-A_16P_TopMnt_Horizontal, symbol Connector:USB_C_Receptacle_USB2.0_16P
- added R12, R13: 5k1, Resistor_SMD:R_0603_1608Metric, symbol Device:R
- added R14, R15: 4k7, Resistor_SMD:R_0603_1608Metric, symbol Device:R
Connections:
- net GND: now also D6.1 (A1), D7.1 (A1), J3.1 (Pin_1), J4.1 (Pin_1), J5.1 (Pin_1), J6.1 (Pin_1), J7.1 (Pin_1), J8.1 (Pin_1), JUARTINV1.A1 (GND), JUARTINV1.A12 (GND), JUARTINV1.B1 (GND), JUARTINV1.B12 (GND), JUARTINV1.S1 (SHIELD), R12.2, R13.2
- net I2C4_SCL_MON: now also J3.2 (Pin_2), R15.1
- net I2C4_SDA_MON: now also J3.3 (Pin_3), R14.2
- net SW_OFFGRID: now also J4.2 (Pin_2)
- net UART1_RX_INV: now also D7.2 (A2), JUARTINV1.A7 (D-), JUARTINV1.B7 (D-); no longer D2.2 (A2)
- net UART1_TX_INV: now also D6.2 (A2), JUARTINV1.A6 (D+), JUARTINV1.B6 (D+); no longer D1.2 (A2)
- net UART6_RX_BMS: now also D2.2 (A2)
- net UART6_TX_BMS: now also D1.2 (A2)
- net VCC_3V: now also JUARTINV1.A4 (VBUS), JUARTINV1.A9 (VBUS), JUARTINV1.B4 (VBUS), JUARTINV1.B9 (VBUS), R14.1, R15.2
- net SW_CHBAT15: now reaches J2.10 (Pin_10)
- net SW_CHBAT15: now also J8.4 (Pin_4)
- net SW_CHBAT10: now reaches J2.11 (Pin_11)
- net SW_CHBAT10: now also J7.3 (Pin_3)
- net SW_CHBAT16: now reaches J2.14 (Pin_14)
- net SW_CHBAT16: now also J8.5 (Pin_5)
- net SW_CHBAT12: now reaches J2.2 (Pin_2)
- net SW_CHBAT12: now also J7.5 (Pin_5)
- net SW_CHBAT13: now reaches J2.4 (Pin_4)
- net SW_CHBAT13: now also J8.2 (Pin_2)
- net SW_CHBAT14: now reaches J2.6 (Pin_6)
- net SW_CHBAT14: now also J8.3 (Pin_3)
- net SW_CHBAT8: now reaches J2.7 (Pin_7)
- net SW_CHBAT8: now also J6.5 (Pin_5)
- net SW_CHBAT9: now reaches J2.9 (Pin_9)
- net SW_CHBAT9: now also J7.2 (Pin_2)
- net SW_CHBAT4: now reaches J1.10 (Pin_10)
- net SW_CHBAT4: now also J5.5 (Pin_5)
- net SW_CHBAT5: now reaches J1.12 (Pin_12)
- net SW_CHBAT5: now also J6.2 (Pin_2)
- net SW_CHBAT6: now reaches J1.13 (Pin_13)
- net SW_CHBAT6: now also J6.3 (Pin_3)
- net SW_CHBAT11: now reaches J1.14 (Pin_14)
- net SW_CHBAT11: now also J7.4 (Pin_4)
- net SW_CHBAT7: now reaches J1.17 (Pin_17)
- net SW_CHBAT7: now also J6.4 (Pin_4)
- net SW_CHBAT1: now reaches J1.5 (Pin_5)
- net SW_CHBAT1: now also J5.2 (Pin_2)
- net SW_CHBAT2: now reaches J1.7 (Pin_7)
- net SW_CHBAT2: now also J5.3 (Pin_3)
- net SW_CHBAT3: now reaches J1.9 (Pin_9)
- net SW_CHBAT3: now also J5.4 (Pin_4)
- new net: JUARTINV1.A5 (CC1), R12.1
- new net: JUARTINV1.B5 (CC2), R13.1
Other:
- note added: "PA15"
- note added: "PA4"
- note added: "PA5"
- note added: "PA6"
- note added: "PA7/PB5"
- note added: "PB1"
- note added: "PB12"
- note added: "PB13"
- note added: "PB5"
- note added: "PC2"
- note added: "PE11"
- note added: "PE13"
- note added: "PE9"
- note added: "PF13"
- note added: "PF4/PA2"
- note added: "PG14/PC4/PG9"
- note added: "PW_USB1_RED"
- note added: "PW_USB2_WHITE_DM"
- note added: "PW_USB3_GREEN_DP"
- note added: "PW_USB4_BLACK"
- moved on the sheet: C1, C3, C5, D4, D5, JCANBMS1, JUARTBMS1, R1, R4, R5, R7, U2
