File: example/nucleo-f767zi_solax-pylontech/pcb/Solax_Pylontech.kicad_sch (KiCad schematic)
At the start: 51 parts, among them J1 Conn_02x10_Odd_Even, J2 Conn_02x07_Odd_Even, J3 Conn_01x03_Socket, J4 Conn_01x02_Socket, J5 Conn_01x05_Socket, J6 Conn_01x05_Socket, J7 Conn_01x05_Socket, J8 Conn_01x05_Socket, U1 LT1107CS, U2 MCP2551-I-SN, U3 MCP2551-I-SN

Commit message: - extract algorithms from the main and have them in separate files for unitary testing - add support for Pylontech SC0500 HV protocol, adapt 2^31 ms fixes - change pcb component from MCP2551 to TAJ1050
Parts:
- U2, U3: value MCP2551-I-SN -> TJA1050 (NOT MCP2551-I-SN)
Changed lines of the file:
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@@
 			)
 		)
-		(property "Value" "MCP2551-I-SN"
+		(property "Value" "TJA1050 (NOT MCP2551-I-SN)"
 			(at 134.0994 71.2271 0)
 			(effects
@@
 			)
 		)
-		(property "Value" "MCP2551-I-SN"
+		(property "Value" "TJA1050 (NOT MCP2551-I-SN)"
 			(at 132.8294 21.6971 0)
 			(effects
